File: twinklr_board.brd (EAGLE design)
At the start: 88 x 32 mm, 27 parts, among them IC1 LM386N-1, IC2 7805TV

Commit message: Making a production board for Ragworm.
Parts:
- removed ENCODER_IN: (no value), pinhead:1X02
- removed JP2: (no value), adafruit:1X01
- added C21: 0.1uF, SparkFun-Capacitors:CPOL-RADIAL-10UF-25V
- added PI_HEADERS: (no value), adafruit:1X03
- C1: value (none) -> 100uF
- C2: value (none) -> 2.2uF
- C20: value (none) -> 0.33uF
- C3: value (none) -> 100nf; device SparkFun-Capacitors:CPOL-RADIAL-10UF-25V -> SparkFun-Capacitors:CAP-PTH-SMALL
- C4: value (none) -> 10uF
- C5: value (none) -> 470uF 20V; device adafruit:B45181A -> SparkFun-Capacitors:CPOL-RADIAL-1000UF-25V
- C6: value (none) -> 47nF; device SparkFun-Capacitors:CPOL-RADIAL-10UF-25V -> SparkFun-Capacitors:AXIAL-5MM
- IC1: value LM386N-1 -> LM386
- IC2: value 7805TV -> 7805
- R1: value (none) -> 10R
- moved C3 30.3 mm to (22.4, 26.6), turned to 270 degrees
- moved C6 28.2 mm to (37.3, 22.5), turned to 270 degrees
- moved C1 27.6 mm to (25.0, 18.5)
- moved C4 27.5 mm to (18.9, 18.2)
- moved R1 25.2 mm to (30.1, 15.5), turned to 90 degrees
- moved C2 16.3 mm to (44.0, 20.0), turned to 0 degrees
- moved ENCODER 14.3 mm to (63.5, 21.4)
- moved R2 10.7 mm to (57.3, 6.96), turned to 270 degrees
- moved POWER 9.60 mm to (54.2, 29.2), turned to 180 degrees
- moved R3 8.81 mm to (54.8, 6.96), turned to 90 degrees
- moved AUDIO 7.38 mm to (54.1, 24.3), turned to 180 degrees
- moved IC1 7.07 mm to (30.5, 25.3)
- moved U$1 6.00 mm to (73.5, 28.5)
- moved U$4 6.00 mm to (73.5, 3.50)
- moved C5 4.78 mm to (43.3, 28.2), turned to 180 degrees
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- renumbered C7 to C20, RV1 to VR1
Connections:
- removed net N$10 (its old number): C5.-, R1.P$2
- removed net N$3 (its old number): C4.2, U$2.P$1
- removed net PIN18: JP2.1, S1.P$1, S1.P$2
- new net N$13: PI_HEADERS.3, S1.P$1, S1.P$2
- new net N$4: C4.1, IC1.1
- new net N$5: C4.2, IC1.8
- net +5V: now also C21.1; no longer C6.1
- net +9V: now also C1.1
- net ENC_A: now also PI_HEADERS.1; no longer ENCODER_IN.1
- net ENC_B: now also PI_HEADERS.2; no longer ENCODER_IN.2
- net GND: now also C1.2, C21.2; no longer C6.2
- net N$1: now also U$2.P$1; no longer C1.1
- net N$2: now also C2.2; no longer C1.2
- net N$6: now also C5.+, C6.P$1, IC1.5; no longer SPEAKER.1, U$2.P$2
- net N$7: now also U$2.P$2; no longer IC1.1
- net N$8: now also C6.P$2, R1.P$2; no longer C2.2, IC1.8
- net N$9: now also C5.-, SPEAKER.1; no longer C4.1, C5.+, IC1.5
Routing:
- net N$13: track 0.00 -> 39.8 mm
- net N$9: track 12.6 -> 39.5 mm
- net N$3 (its old number): track 18.6 -> 0.00 mm
- net N$5: track 0.00 -> 18.5 mm
- net PIN18: track 16.3 -> 0.00 mm
- net N$1: track 10.4 -> 24.3 mm
- net N$10: track 20.3 -> 7.87 mm
- net ENC_B: track 27.2 -> 17.8 mm
- net N$4: track 0.00 -> 8.08 mm
- net N$2: track 13.8 -> 6.00 mm
- net +9V: track 61.1 -> 54.1 mm
- net +5V: track 124.2 -> 118.8 mm
- net N$6: track 13.1 -> 9.68 mm
- net N$10 (its old number): track 2.90 -> 0.00 mm
- net N$3: track 5.88 -> 7.89 mm
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- added copper zone on layer 16, net GND
- removed copper zone on layer 16, net N$12
Other:
- board size 88 x 32 mm -> 83 x 32 mm
- board text added: "17"
- board text added: "18"
- board text added: "27"
- board text added: "Twinklr Main Board v1.01 tom@infovore.org"
- board text removed: "Twinklr Main Board v1.00 tom@infovore.org"

Commit message: Yanking out audio ground.
Connections:
- new net AUDIOGND: AUDIO.2, U$2.P$3
- net GND: no longer AUDIO.2, U$2.P$3
Changed lines of the file:
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@@
 <contactref element="S1" pad="P$3"/>
 <contactref element="S1" pad="P$4"/>
-<contactref element="U$2" pad="P$3"/>
-<contactref element="AUDIO" pad="2"/>
 <contactref element="SPEAKER" pad="2"/>
 <contactref element="R1" pad="P$1"/>
@@
 <vertex x="-3" y="32" curve="90"/>
 </polygon>
+<wire x1="63.3856125" y1="16.193953125" x2="52.95391875" y2="29.24913125" width="0" layer="19" extent="1-1"/>
+<wire x1="63.450190625" y1="4.9963" x2="63.3856125" y2="16.193953125" width="0" layer="19" extent="1-1"/>
+<wire x1="34.350828125" y1="21.4758375" x2="52.95391875" y2="29.24913125" width="0" layer="19" extent="1-1"/>
+<wire x1="29.270828125" y1="21.4758375" x2="34.350828125" y2="21.4758375" width="0" layer="19" extent="1-1"/>
+<wire x1="34.02108125" y1="15.540671875" x2="34.350828125" y2="21.4758375" width="0" layer="19" extent="1-1"/>
+<wire x1="30.063690625" y1="11.739871875" x2="34.02108125" y2="15.540671875" width="0" layer="19" extent="1-1"/>
+<wire x1="23.68546875" y1="18.478121875" x2="29.270828125" y2="21.4758375" width="0" layer="19" extent="1-1"/>
+<wire x1="22.439671875" y1="24.05176875" x2="23.68546875" y2="18.478121875" width="0" layer="19" extent="1-1"/>
+<wire x1="26.5" y1="5.814778125" x2="30.063690625" y2="11.739871875" width="0" layer="19" extent="1-1"/>
+<wire x1="21.5" y1="5.814778125" x2="26.5" y2="5.814778125" width="0" layer="19" extent="1-1"/>
+<wire x1="14.49273125" y1="4.45873125" x2="21.5" y2="5.814778125" width="0" layer="19" extent="1-1"/>
+<wire x1="14.37493125" y1="11.678203125" x2="14.49273125" y2="4.45873125" width="0" layer="19" extent="1-1"/>
+<wire x1="3.5" y1="8.7" x2="14.37493125" y2="11.678203125" width="0" layer="19" extent="1-1"/>
+<wire x1="8.158959375" y1="28.272571875" x2="22.439671875" y2="24.05176875" width="0" layer="19" extent="1-1"/>
 </signal>
 <signal name="+9V">
@@
 <wire x1="45.27286875" y1="19.99713125" x2="45.27" y2="20" width="0.4064" layer="16"/>
 </signal>
+<signal name="AUDIOGND">
+<contactref element="AUDIO" pad="2"/>
+<contactref element="U$2" pad="P$3"/>
+<wire x1="48.83" y1="15.39" x2="52.8200375" y2="24.307759375" width="0" layer="19" extent="1-1"/>
+</signal>
 </signals>
