File: twinklr_board.sch (EAGLE design)
At the start: 23 parts, among them IC1 LM386N-1, IC2 7805TV

Commit message: Making a production board for Ragworm.
Parts:
- removed ENCODER_IN: (no value), pinhead:PINHD-1X2
- removed JP2: (no value), adafruit:PINHD-1X1
- added C21: 0.1uF, SparkFun-Capacitors:CAP_POLPTH2
- added PI_HEADERS: (no value), adafruit:PINHD-1X3
- C1: value (none) -> 100uF
- C2: value (none) -> 2.2uF
- C20: value (none) -> 0.33uF
- C3: value (none) -> 100nf; device SparkFun-Capacitors:CAP_POLPTH2 -> SparkFun-Capacitors:CAPPTH
- C4: value (none) -> 10uF
- C5: value (none) -> 470uF 20V; device adafruit:CPOL-USB45181A -> SparkFun-Capacitors:CAP_POLPTH4
- C6: value (none) -> 47nF; device SparkFun-Capacitors:CAP_POLPTH2 -> SparkFun-Capacitors:CAP_
- IC1: value LM386N-1 -> LM386
- IC2: value 7805TV -> 7805
- R1: value (none) -> 10R
- renumbered C7 to C20, RV1 to VR1
Connections:
- removed net N$3 (its old number): C4.-, U$2.2
- removed net PIN18: JP2.1, S1.O
- new net N$13: PI_HEADERS.3, S1.O
- new net N$4: C4.+, IC1.GAIN@1
- net +5V: now also C21.+; no longer C6.+
- net +9V: now also C1.+
- net ENC_A: now also PI_HEADERS.1; no longer ENCODER_IN.1
- net ENC_B: now also PI_HEADERS.2; no longer ENCODER_IN.2
- net GND: now also C1.-, C21.-, C3.2; no longer C3.-, C6.-
- net N$1: now also U$2.2; no longer C1.+
- net N$10: now also C3.1, IC1.BYPASS; no longer C5.-, R1.2
- net N$2: now also C2.-; no longer C1.-
- net N$5: now also C4.-, IC1.GAIN@2; no longer C3.+, IC1.BYPASS
- net N$6: now also C5.+, C6.1, IC1.OUT; no longer SPEAKER-1.K, U$2.3
- net N$7: now also U$2.3; no longer IC1.GAIN@1
- net N$8: now also C6.2, R1.2; no longer C2.-, IC1.GAIN@2
- net N$9: now also C5.-, SPEAKER-1.K; no longer C4.+, C5.+, IC1.OUT
Other:
- moved on the sheet: C1, C2, C4, C5, R1, S1, U$2

Commit message: Yanking out audio ground.
Connections:
- new net AUDIOGND: AUDIO.2, U$2.1
- net GND: no longer AUDIO.2, U$2.1
Changed lines of the file:
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@@
 </classes>
 <parts>
-<part name="SUPPLY1" library="supply2" deviceset="GND" device=""/>
 <part name="IC1" library="linear" deviceset="LM386?-*" device="N" technology="1" value="LM386"/>
 <part name="SUPPLY2" library="supply2" deviceset="GND" device=""/>
@@
 <part name="U$2" library="thonkiconn" deviceset="WQP-PJ301M-12_JACK" device=""/>
 <part name="SPEAKER" library="con-phoenix-350" deviceset="1751248" device=""/>
-<part name="SUPPLY6" library="supply2" deviceset="GND" device=""/>
 <part name="AUDIO" library="pinhead" deviceset="PINHD-1X2" device=""/>
 <part name="JP1" library="foxfield" deviceset="POWER_JACK_VERT" device=""/>
@@
 </plain>
 <instances>
-<instance part="SUPPLY1" gate="GND" x="17.78" y="53.34"/>
 <instance part="IC1" gate="G$1" x="60.96" y="76.2"/>
 <instance part="SUPPLY2" gate="GND" x="48.26" y="71.12"/>
@@
 <instance part="SPEAKER" gate="-1" x="119.38" y="76.2"/>
 <instance part="SPEAKER" gate="-2" x="119.38" y="68.58"/>
-<instance part="SUPPLY6" gate="GND" x="22.86" y="83.82"/>
 <instance part="AUDIO" gate="G$1" x="7.62" y="71.12" rot="MR0"/>
 <instance part="JP1" gate="G$1" x="25.4" y="12.7" rot="MR180"/>
@@
 </segment>
 <segment>
-<pinref part="U$2" gate="G$1" pin="1"/>
-<pinref part="SUPPLY6" gate="GND" pin="GND"/>
-<wire x1="22.86" y1="88.9" x2="22.86" y2="86.36" width="0.1524" layer="91"/>
-</segment>
-<segment>
-<pinref part="AUDIO" gate="G$1" pin="2"/>
-<pinref part="SUPPLY1" gate="GND" pin="GND"/>
-<wire x1="10.16" y1="71.12" x2="17.78" y2="71.12" width="0.1524" layer="91"/>
-<wire x1="17.78" y1="71.12" x2="17.78" y2="55.88" width="0.1524" layer="91"/>
-</segment>
-<segment>
 <pinref part="C1" gate="G$1" pin="-"/>
 <pinref part="SUPPLY8" gate="GND" pin="GND"/>
@@
 </segment>
 </net>
+<net name="AUDIOGND" class="0">
+<segment>
+<pinref part="AUDIO" gate="G$1" pin="2"/>
+<wire x1="10.16" y1="71.12" x2="17.78" y2="71.12" width="0.1524" layer="91"/>
+<wire x1="17.78" y1="71.12" x2="17.78" y2="55.88" width="0.1524" layer="91"/>
+<label x="17.78" y="55.88" size="1.27" layer="95" xref="yes"/>
+</segment>
+<segment>
+<pinref part="U$2" gate="G$1" pin="1"/>
+<wire x1="22.86" y1="88.9" x2="22.86" y2="86.36" width="0.1524" layer="91"/>
+<label x="22.86" y="86.36" size="1.27" layer="95" xref="yes"/>
+</segment>
+</net>
